Commit message: 1.1.5.20241118092402

File: resources/robots/pointfoot/WF_TRON1A/urdf/robot.urdf (robot description, URDF)
Before this commit: robot wheel_biped, 9 links, 8 joints
Links:
- added link limx_imu, mass 0.01; visual box size=0.015 0.015 0.004
- link base_Link: geometry collision box size=0.37 0.26 0.14; visual mesh filename=../meshes/base_Link.STL
- link wheel_L_Link: geometry collision cylinder length=0.017 radius=0.127; visual mesh filename=../meshes/wheel_L_Link.STL
- link wheel_R_Link: geometry collision cylinder length=0.017 radius=0.127; visual mesh filename=../meshes/wheel_R_Link.STL
Joints:
- added joint limx_imu_joint: type fixed, parent base_Link, child limx_imu, origin xyz=0. 0. 0. rpy=0. 0. 0.
- joint wheel_L_Joint: limit lower=-1000000 upper=1000000 effort=40 velocity=40 -> lower=-100000 upper=100000 effort=40 velocity=40
- joint wheel_R_Joint: limit lower=-1000000 upper=1000000 effort=40 velocity=40 -> lower=-100000 upper=100000 effort=40 velocity=40
