Commit message: 1.1.5.20250217163732

File: resources/robots/pointfoot/PF_P441A/urdf/robot.urdf (robot description, URDF)
Before this commit: robot point_foot, 12 links, 11 joints
Links:
- link abad_L_Link: geometry collision cylinder length=0.05 radius=0.05; visual mesh filename=../meshes/abad_L_Link.STL
- link abad_R_Link: geometry collision cylinder length=0.05 radius=0.05; visual mesh filename=../meshes/abad_R_Link.STL
- link base_Link: geometry collision box size=0.37 0.26 0.14; visual mesh filename=../meshes/base_Link.STL
- link foot_L_Link: geometry collision sphere radius=0.032; visual mesh filename=../meshes/foot_L_Link.STL
- link foot_R_Link: geometry collision sphere radius=0.032; visual mesh filename=../meshes/foot_R_Link.STL
- link hip_L_Link: geometry collision cylinder length=0.15 radius=0.035; visual mesh filename=../meshes/hip_L_Link.STL
- link hip_R_Link: geometry collision cylinder length=0.15 radius=0.035; visual mesh filename=../meshes/hip_R_Link.STL
- link knee_L_Link: geometry collision cylinder length=0.26 radius=0.015; visual mesh filename=../meshes/knee_L_Link.STL
- link knee_R_Link: geometry collision cylinder length=0.26 radius=0.015; visual mesh filename=../meshes/knee_R_Link.STL

File: resources/robots/pointfoot/PF_P441B/urdf/robot.urdf (robot description, URDF)
Before this commit: robot point_foot, 12 links, 11 joints
Links:
- link abad_L_Link: geometry collision cylinder length=0.05 radius=0.05; visual mesh filename=../meshes/abad_L_Link.STL
- link abad_R_Link: geometry collision cylinder length=0.05 radius=0.05; visual mesh filename=../meshes/abad_R_Link.STL
- link base_Link: geometry collision box size=0.28 0.24 0.14; visual mesh filename=../meshes/base_Link.STL
- link foot_L_Link: geometry collision sphere radius=0.032; visual mesh filename=../meshes/foot_L_Link.STL
- link foot_R_Link: geometry collision sphere radius=0.032; visual mesh filename=../meshes/foot_R_Link.STL
- link hip_L_Link: geometry collision cylinder length=0.15 radius=0.025; visual mesh filename=../meshes/hip_L_Link.STL
- link hip_R_Link: geometry collision cylinder length=0.15 radius=0.025; visual mesh filename=../meshes/hip_R_Link.STL
- link knee_L_Link: geometry collision cylinder length=0.26 radius=0.015; visual mesh filename=../meshes/knee_L_Link.STL
- link knee_R_Link: geometry collision cylinder length=0.26 radius=0.015; visual mesh filename=../meshes/knee_R_Link.STL

File: resources/robots/pointfoot/PF_P441C/urdf/robot.urdf (robot description, URDF)
Before this commit: robot point_foot, 12 links, 11 joints
Links:
- link abad_L_Link: geometry collision cylinder length=0.05 radius=0.05; visual mesh filename=../meshes/abad_L_Link.STL
- link abad_R_Link: geometry collision cylinder length=0.05 radius=0.05; visual mesh filename=../meshes/abad_R_Link.STL
- link base_Link: geometry collision box size=0.25 0.26 0.18; visual mesh filename=../meshes/base_Link.STL
- link foot_L_Link: geometry collision sphere radius=0.032; visual mesh filename=../meshes/foot_L_Link.STL
- link foot_R_Link: geometry collision sphere radius=0.032; visual mesh filename=../meshes/foot_R_Link.STL
- link hip_L_Link: geometry collision cylinder length=0.18 radius=0.035; visual mesh filename=../meshes/hip_L_Link.STL
- link hip_R_Link: geometry collision cylinder length=0.18 radius=0.035; visual mesh filename=../meshes/hip_R_Link.STL
- link knee_L_Link: geometry collision cylinder length=0.26 radius=0.015; visual mesh filename=../meshes/knee_L_Link.STL
- link knee_R_Link: geometry collision cylinder length=0.26 radius=0.015; visual mesh filename=../meshes/knee_R_Link.STL

File: resources/robots/pointfoot/PF_P441C2/urdf/robot.urdf (robot description, URDF)
Before this commit: robot point_foot, 12 links, 11 joints
Links:
- link abad_L_Link: geometry collision cylinder length=0.05 radius=0.05; visual mesh filename=../meshes/abad_L_Link.STL
- link abad_R_Link: geometry collision cylinder length=0.05 radius=0.05; visual mesh filename=../meshes/abad_R_Link.STL
- link base_Link: geometry collision box size=0.265 0.26 0.18; visual mesh filename=../meshes/base_Link.STL
- link foot_L_Link: geometry collision sphere radius=0.032; visual mesh filename=../meshes/foot_L_Link.STL
- link foot_R_Link: geometry collision sphere radius=0.032; visual mesh filename=../meshes/foot_R_Link.STL
- link hip_L_Link: geometry collision cylinder length=0.18 radius=0.035; visual mesh filename=../meshes/hip_L_Link.STL
- link hip_R_Link: geometry collision cylinder length=0.18 radius=0.035; visual mesh filename=../meshes/hip_R_Link.STL
- link knee_L_Link: geometry collision cylinder length=0.26 radius=0.015; visual mesh filename=../meshes/knee_L_Link.STL
- link knee_R_Link: geometry collision cylinder length=0.26 radius=0.015; visual mesh filename=../meshes/knee_R_Link.STL

File: resources/robots/pointfoot/PF_TRON1A/urdf/robot.urdf (robot description, URDF)
Before this commit: robot point_foot, 12 links, 11 joints
Links:
- link abad_L_Link: geometry collision cylinder length=0.05 radius=0.05; visual mesh filename=../meshes/abad_L_Link.STL
- link abad_R_Link: geometry collision cylinder length=0.05 radius=0.05; visual mesh filename=../meshes/abad_R_Link.STL
- link base_Link: geometry collision box size=0.265 0.26 0.18; visual mesh filename=../meshes/base_Link.STL
- link foot_L_Link: geometry collision sphere radius=0.032; visual mesh filename=../meshes/foot_L_Link.STL
- link foot_R_Link: geometry collision sphere radius=0.032; visual mesh filename=../meshes/foot_R_Link.STL
- link hip_L_Link: geometry collision cylinder length=0.18 radius=0.035; visual mesh filename=../meshes/hip_L_Link.STL
- link hip_R_Link: geometry collision cylinder length=0.18 radius=0.035; visual mesh filename=../meshes/hip_R_Link.STL
- link knee_L_Link: geometry collision cylinder length=0.26 radius=0.015; visual mesh filename=../meshes/knee_L_Link.STL
- link knee_R_Link: geometry collision cylinder length=0.26 radius=0.015; visual mesh filename=../meshes/knee_R_Link.STL

File: resources/robots/pointfoot/SF_TRON1A/urdf/robot.urdf (robot description, URDF)
Before this commit: robot SF_TRON1, 10 links, 9 joints
Links:
- link abad_L_Link: geometry collision cylinder length=0.05 radius=0.05; visual mesh filename=../meshes/abad_L_Link.STL
- link abad_R_Link: geometry collision cylinder length=0.05 radius=0.05; visual mesh filename=../meshes/abad_R_Link.STL
- link ankle_L_Link: geometry collision mesh filename=../meshes/ankle_L_Link.STL; visual mesh filename=../meshes/ankle_L_Link.STL
- link ankle_R_Link: geometry collision mesh filename=../meshes/ankle_R_Link.STL; visual mesh filename=../meshes/ankle_R_Link.STL
- link base_Link: geometry collision box size=0.27 0.26 0.19; visual mesh filename=../meshes/base_Link.STL
- link hip_L_Link: geometry collision cylinder length=0.15 radius=0.035; visual mesh filename=../meshes/hip_L_Link.STL
- link hip_R_Link: geometry collision cylinder length=0.15 radius=0.035; visual mesh filename=../meshes/hip_R_Link.STL
- link knee_L_Link: geometry collision cylinder length=0.26 radius=0.02; visual mesh filename=../meshes/knee_L_Link.STL
- link knee_R_Link: geometry collision cylinder length=0.26 radius=0.02; visual mesh filename=../meshes/knee_R_Link.STL

File: resources/robots/pointfoot/WF_TRON1A/urdf/robot.urdf (robot description, URDF)
Before this commit: robot wheel_biped, 10 links, 9 joints
Links:
- link abad_L_Link: geometry collision cylinder length=0.05 radius=0.05; visual mesh filename=../meshes/abad_L_Link.STL
- link abad_R_Link: geometry collision cylinder length=0.05 radius=0.05; visual mesh filename=../meshes/abad_R_Link.STL
- link base_Link: geometry collision box size=0.27 0.26 0.19; visual mesh filename=../meshes/base_Link.STL
- link hip_L_Link: geometry collision cylinder length=0.15 radius=0.035; visual mesh filename=../meshes/hip_L_Link.STL
- link hip_R_Link: geometry collision cylinder length=0.15 radius=0.035; visual mesh filename=../meshes/hip_R_Link.STL
- link knee_L_Link: geometry collision cylinder length=0.26 radius=0.015; visual mesh filename=../meshes/knee_L_Link.STL
- link knee_R_Link: geometry collision cylinder length=0.26 radius=0.015; visual mesh filename=../meshes/knee_R_Link.STL
- link wheel_L_Link: geometry collision cylinder length=0.05 radius=0.127; visual mesh filename=../meshes/wheel_L_Link.STL
- link wheel_R_Link: geometry collision cylinder length=0.05 radius=0.127; visual mesh filename=../meshes/wheel_R_Link.STL
